File: psu.brd (EAGLE design)
At the start: 94.9 x 63.5 mm, 27 parts, among them IC1 7809, IC2 7909

Commit message: Routed!
Parts:
- moved D10 3.81 mm to (59.7, 34.3), turned to 180 degrees
- turned C4 to 180 degrees
- turned C6 to 270 degrees
- turned D12 to 180 degrees
Connections:
- net OUT_NEG: now also JP3.1; no longer JP3.3
- net OUT_POS: now also JP3.3; no longer JP3.1
Routing:
- net N$8: track 0.00 -> 170.9 mm
- net GND: track 188.5 -> 314.1 mm
- net OUT_NEG: track 0.00 -> 45.6 mm
- net OUT_POS: track 64.8 -> 53.4 mm
- net IN2_AC_B: track 13.0 -> 19.4 mm
