File: psu.brd (EAGLE design)
At the start: 94.9 x 63.5 mm, 27 parts, among them IC1 7809, IC2 7909

Commit message: wip
Parts:
- moved C3 30.7 mm to (69.8, 67.3), turned to 180 degrees
- moved C4 30.1 mm to (69.8, 31.8), turned to 0 degrees
- moved C5 6.84 mm to (69.8, 62.2), turned to 0 degrees
- moved C6 5.68 mm to (69.8, 35.6), turned to 0 degrees
- moved C2 5.24 mm to (41.9, 39.4)
- moved C1 4.02 mm to (41.9, 59.7)
- moved D10 3.81 mm to (59.7, 38.1)
- moved D9 2.54 mm to (59.7, 58.4)
- moved IC1 1.27 mm to (71.1, 72.4), turned to 180 degrees
- moved KK1 1.27 mm to (71.1, 72.4), turned to 0 degrees
- turned IC2 to 0 degrees
- turned KK2 to 180 degrees
Routing:
- net GND: track 315.3 -> 272.7 mm
- net N$8: track 172.5 -> 141.7 mm
- net OUT_POS: track 53.4 -> 75.0 mm
- net N$1: track 82.5 -> 102.3 mm
- net OUT_NEG: track 45.6 -> 59.6 mm
Other:
- board size 94.9 x 63.5 mm -> 94.9 x 64.8 mm

Commit message: wip
Parts:
- moved C3 2.54 mm to (72.4, 67.3)
- turned D12 to 0 degrees
Connections:
- net GND: now also D12.C; no longer D12.A
- net OUT_NEG: now also D12.A; no longer D12.C
Routing:
- net GND: track 272.7 -> 270.6 mm
- net OUT_POS: track 75.0 -> 72.9 mm
- net N$1: track 102.3 -> 101.3 mm
- added copper zone on layer 16, net GND
Other:
- board text added: "+9V"
- board text added: "-9V"
- board text added: "GND"
- board text added: "badcircuits.ru"
Changed lines of the file:
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@@
 <hole x="91.44" y="20.32" drill="2.8"/>
 <hole x="91.44" y="77.47" drill="2.8"/>
+<text x="87.63" y="53.34" size="1.016" layer="16" font="vector" rot="MR0">+9V</text>
+<text x="87.63" y="44.45" size="1.016" layer="16" font="vector" rot="MR0">-9V</text>
+<text x="87.63" y="50.8" size="1.016" layer="16" font="vector" rot="MR0">GND</text>
+<text x="48.26" y="78.74" size="1.016" layer="16" font="vector" rot="MR0">badcircuits.ru</text>
 </plain>
 <attributes>
@@
 <element name="C1" library="rcl" package="E7,5-18" value="10000uF" x="41.91" y="59.69"/>
 <element name="C2" library="rcl" package="E7,5-18" value="10000uF" x="41.91" y="39.37"/>
-<element name="C3" library="rcl" package="C025-025X050" value="100nF" x="69.85" y="67.31" rot="R180"/>
+<element name="C3" library="rcl" package="C025-025X050" value="100nF" x="72.39" y="67.31" rot="R180"/>
 <element name="C4" library="rcl" package="C025-025X050" value="100nF" x="69.85" y="31.75"/>
 <element name="C5" library="rcl" package="C025-025X050" value="100nF" x="69.85" y="62.23"/>
@@
 <element name="D10" library="diode" package="DO41-10" value="1N4007" x="59.69" y="38.1" rot="R180"/>
 <element name="D11" library="diode" package="DO41-10" value="1N4007" x="59.69" y="53.34"/>
-<element name="D12" library="diode" package="DO41-10" value="1N4007" x="59.69" y="43.18" rot="R180"/>
+<element name="D12" library="diode" package="DO41-10" value="1N4007" x="59.69" y="43.18"/>
 <element name="D2" library="diode" package="DO201-15" value="1N5821" x="21.59" y="67.31" rot="R180"/>
 <element name="D3" library="diode" package="DO201-15" value="1N5821" x="21.59" y="60.96"/>
@@
 <wire x1="72.39" y1="78.74" x2="73.66" y2="77.47" width="1.016" layer="16"/>
 <wire x1="73.66" y1="77.47" x2="73.66" y2="74.93" width="1.016" layer="16"/>
-<wire x1="71.12" y1="67.31" x2="73.66" y2="69.85" width="1.016" layer="16"/>
-<wire x1="73.66" y1="69.85" x2="73.66" y2="74.93" width="1.016" layer="16"/>
+<wire x1="73.66" y1="67.31" x2="73.66" y2="74.93" width="1.016" layer="16"/>
 <wire x1="54.61" y1="74.93" x2="58.42" y2="78.74" width="1.016" layer="16"/>
 <wire x1="58.42" y1="78.74" x2="72.39" y2="78.74" width="1.016" layer="16"/>
@@
 <wire x1="64.77" y1="58.42" x2="66.04" y2="57.15" width="1.016" layer="16"/>
 <wire x1="66.04" y1="57.15" x2="80.01" y2="57.15" width="1.016" layer="16"/>
-<wire x1="68.58" y1="62.23" x2="66.04" y2="64.77" width="1.016" layer="16"/>
-<wire x1="66.04" y1="64.77" x2="66.04" y2="68.58" width="1.016" layer="16"/>
-<wire x1="66.04" y1="68.58" x2="68.58" y2="71.12" width="1.016" layer="16"/>
-<wire x1="68.58" y1="71.12" x2="68.58" y2="74.93" width="1.016" layer="16"/>
+<wire x1="68.58" y1="74.93" x2="68.58" y2="62.23" width="1.016" layer="16"/>
 </signal>
 <signal name="OUT_NEG">
@@
 <contactref element="C8" pad="-"/>
 <contactref element="D10" pad="C"/>
-<contactref element="D12" pad="C"/>
 <contactref element="JP3" pad="1"/>
 <wire x1="80.01" y1="39.37" x2="87.63" y2="39.37" width="1.016" layer="16"/>
@@
 <wire x1="87.63" y1="39.37" x2="90.17" y2="41.91" width="1.016" layer="16"/>
 <wire x1="90.17" y1="41.91" x2="90.17" y2="44.45" width="1.016" layer="16"/>
-<wire x1="64.77" y1="43.18" x2="64.77" y2="38.1" width="1.016" layer="16"/>
 <wire x1="73.66" y1="24.13" x2="76.2" y2="26.67" width="1.016" layer="16"/>
 <wire x1="76.2" y1="26.67" x2="76.2" y2="39.37" width="1.016" layer="16"/>
@@
 <wire x1="71.12" y1="36.83" x2="69.85" y2="38.1" width="1.016" layer="16"/>
 <wire x1="69.85" y1="38.1" x2="64.77" y2="38.1" width="1.016" layer="16"/>
+<contactref element="D12" pad="A"/>
+<wire x1="64.77" y1="43.18" x2="64.77" y2="38.1" width="1.016" layer="16"/>
 </signal>
 <signal name="IN2_AC_A">
@@
 <contactref element="D5" pad="C"/>
 <contactref element="D6" pad="C"/>
-<contactref element="D12" pad="A"/>
 <contactref element="JP3" pad="2"/>
 <wire x1="90.17" y1="49.45" x2="90.09" y2="49.53" width="1.016" layer="16"/>
@@
 <wire x1="36.83" y1="53.34" x2="36.83" y2="49.53" width="1.016" layer="16"/>
 <wire x1="64.77" y1="53.34" x2="64.77" y2="49.53" width="1.016" layer="16"/>
-<wire x1="54.61" y1="43.18" x2="54.61" y2="49.53" width="1.016" layer="16"/>
 <wire x1="29.21" y1="25.4" x2="25.4" y2="25.4" width="1.016" layer="16"/>
 <wire x1="25.4" y1="25.4" x2="24.13" y2="26.67" width="1.016" layer="16"/>
@@
 <wire x1="68.58" y1="24.13" x2="59.69" y2="33.02" width="1.016" layer="16"/>
 <wire x1="59.69" y1="33.02" x2="59.69" y2="36.83" width="1.016" layer="16"/>
-<wire x1="59.69" y1="36.83" x2="54.61" y2="41.91" width="1.016" layer="16"/>
-<wire x1="54.61" y1="41.91" x2="54.61" y2="43.18" width="1.016" layer="16"/>
-<wire x1="71.12" y1="74.93" x2="71.12" y2="71.12" width="1.016" layer="16"/>
-<wire x1="71.12" y1="71.12" x2="68.58" y2="68.58" width="1.016" layer="16"/>
-<wire x1="68.58" y1="68.58" x2="68.58" y2="67.31" width="1.016" layer="16"/>
 <wire x1="68.58" y1="31.75" x2="68.58" y2="24.13" width="1.016" layer="16"/>
 <wire x1="29.21" y1="38.1" x2="34.29" y2="38.1" width="1.016" layer="16"/>
@@
 <wire x1="45.72" y1="59.69" x2="45.72" y2="49.53" width="1.016" layer="16"/>
 <wire x1="68.58" y1="35.56" x2="68.58" y2="31.75" width="1.016" layer="16"/>
-<wire x1="71.12" y1="62.23" x2="71.12" y2="63.5" width="1.016" layer="16"/>
-<wire x1="71.12" y1="63.5" x2="68.58" y2="66.04" width="1.016" layer="16"/>
-<wire x1="68.58" y1="66.04" x2="68.58" y2="67.31" width="1.016" layer="16"/>
 <wire x1="71.12" y1="62.23" x2="72.39" y2="60.96" width="1.016" layer="16"/>
 <wire x1="72.39" y1="60.96" x2="90.17" y2="60.96" width="1.016" layer="16"/>
@@
 <wire x1="92.71" y1="52.07" x2="90.17" y2="49.53" width="1.016" layer="16"/>
 <wire x1="90.17" y1="49.53" x2="90.17" y2="49.45" width="1.016" layer="16"/>
+<wire x1="71.12" y1="74.93" x2="71.12" y2="67.31" width="1.016" layer="16"/>
+<wire x1="71.12" y1="67.31" x2="71.12" y2="62.23" width="1.016" layer="16"/>
+<polygon width="0.254" layer="16" spacing="2.54" pour="hatch" isolate="1.27">
+<vertex x="1.27" y="80.01"/>
+<vertex x="25.4" y="80.01"/>
+<vertex x="25.4" y="74.93"/>
+<vertex x="63.5" y="74.93"/>
+<vertex x="63.5" y="80.01"/>
+<vertex x="93.98" y="80.01"/>
+<vertex x="93.98" y="17.78"/>
+<vertex x="1.27" y="17.78"/>
+</polygon>
+<contactref element="D12" pad="C"/>
+<wire x1="54.61" y1="43.18" x2="54.61" y2="49.53" width="1.016" layer="16"/>
+<wire x1="54.61" y1="43.18" x2="54.61" y2="41.91" width="1.016" layer="16"/>
+<wire x1="54.61" y1="41.91" x2="59.69" y2="36.83" width="1.016" layer="16"/>
 </signal>
 </signals>
