File: psu.sch (EAGLE design)
At the start: 27 parts, among them IC1 7809, IC2 7909

Commit message: Routed!
Connections:
- net OUT_NEG: now also JP3.1; no longer JP3.3
- net OUT_POS: now also JP3.3; no longer JP3.1
Other:
- moved on the sheet: JP3
Changed lines of the file:
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@@
 <instance part="JP1" gate="G$1" x="-78.74" y="27.94"/>
 <instance part="JP2" gate="G$1" x="-78.74" y="-20.32"/>
-<instance part="JP3" gate="G$1" x="63.5" y="2.54" rot="R180"/>
+<instance part="JP3" gate="G$1" x="63.5" y="2.54" rot="MR0"/>
 <instance part="GND3" gate="1" x="48.26" y="0"/>
 <instance part="KK1" gate="G$1" x="12.7" y="45.72"/>
@@
 <wire x1="15.24" y1="58.42" x2="25.4" y2="58.42" width="0.1524" layer="91"/>
 <wire x1="25.4" y1="58.42" x2="25.4" y2="35.56" width="0.1524" layer="91"/>
-<pinref part="JP3" gate="G$1" pin="1"/>
+<pinref part="D11" gate="1" pin="C"/>
+<pinref part="JP3" gate="G$1" pin="3"/>
 <wire x1="55.88" y1="5.08" x2="55.88" y2="35.56" width="0.1524" layer="91"/>
 <wire x1="55.88" y1="35.56" x2="45.72" y2="35.56" width="0.1524" layer="91"/>
 <junction x="45.72" y="35.56"/>
-<pinref part="D11" gate="1" pin="C"/>
 </segment>
 </net>
@@
 <wire x1="15.24" y1="-53.34" x2="25.4" y2="-53.34" width="0.1524" layer="91"/>
 <wire x1="25.4" y1="-53.34" x2="25.4" y2="-33.02" width="0.1524" layer="91"/>
-<pinref part="JP3" gate="G$1" pin="3"/>
+<pinref part="D12" gate="1" pin="C"/>
+<pinref part="JP3" gate="G$1" pin="1"/>
 <wire x1="55.88" y1="0" x2="55.88" y2="-33.02" width="0.1524" layer="91"/>
 <wire x1="55.88" y1="-33.02" x2="45.72" y2="-33.02" width="0.1524" layer="91"/>
 <junction x="45.72" y="-33.02"/>
-<pinref part="D12" gate="1" pin="C"/>
 </segment>
 </net>

Commit message: wip
Connections:
- net GND: now also D12.C; no longer D12.A
- net OUT_NEG: now also D12.A; no longer D12.C
Other:
- moved on the sheet: D12
Changed lines of the file:
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@@
 <attribute name="VALUE" x="55.6514" y="23.622" size="1.778" layer="96" rot="R180"/>
 </instance>
-<instance part="D12" gate="1" x="45.72" y="-24.13" smashed="yes" rot="R270">
-<attribute name="NAME" x="46.2026" y="-21.59" size="1.778" layer="95"/>
-<attribute name="VALUE" x="45.9486" y="-29.21" size="1.778" layer="96"/>
+<instance part="D12" gate="1" x="45.72" y="-22.86" smashed="yes" rot="R90">
+<attribute name="NAME" x="52.8574" y="-22.86" size="1.778" layer="95" rot="R180"/>
+<attribute name="VALUE" x="55.6514" y="-25.4" size="1.778" layer="96" rot="R180"/>
 </instance>
 <instance part="C1" gate="G$1" x="-12.7" y="25.4"/>
@@
 <wire x1="20.32" y1="-33.02" x2="25.4" y2="-33.02" width="0.1524" layer="91"/>
 <wire x1="25.4" y1="-33.02" x2="35.56" y2="-33.02" width="0.1524" layer="91"/>
-<wire x1="35.56" y1="-33.02" x2="45.72" y2="-33.02" width="0.1524" layer="91"/>
-<wire x1="45.72" y1="-33.02" x2="45.72" y2="-26.67" width="0.1524" layer="91"/>
 <pinref part="C6" gate="G$1" pin="2"/>
-<wire x1="45.72" y1="-26.67" x2="45.72" y2="-25.4" width="0.1524" layer="91"/>
 <wire x1="25.4" y1="-27.94" x2="25.4" y2="-33.02" width="0.1524" layer="91"/>
 <junction x="25.4" y="-33.02"/>
@@
 <wire x1="15.24" y1="-53.34" x2="25.4" y2="-53.34" width="0.1524" layer="91"/>
 <wire x1="25.4" y1="-53.34" x2="25.4" y2="-33.02" width="0.1524" layer="91"/>
-<pinref part="D12" gate="1" pin="C"/>
 <pinref part="JP3" gate="G$1" pin="1"/>
 <wire x1="55.88" y1="0" x2="55.88" y2="-33.02" width="0.1524" layer="91"/>
 <wire x1="55.88" y1="-33.02" x2="45.72" y2="-33.02" width="0.1524" layer="91"/>
+<pinref part="D12" gate="1" pin="A"/>
+<wire x1="45.72" y1="-33.02" x2="35.56" y2="-33.02" width="0.1524" layer="91"/>
+<wire x1="45.72" y1="-25.4" x2="45.72" y2="-33.02" width="0.1524" layer="91"/>
 <junction x="45.72" y="-33.02"/>
 </segment>
@@
 <wire x1="45.72" y1="12.7" x2="45.72" y2="23.622" width="0.1524" layer="91"/>
 <pinref part="C1" gate="G$1" pin="-"/>
-<wire x1="45.72" y1="23.622" x2="45.72" y2="25.4" width="0.1524" layer="91"/>
 <wire x1="-12.7" y1="20.32" x2="-12.7" y2="12.7" width="0.1524" layer="91"/>
 <junction x="-12.7" y="12.7"/>
@@
 <junction x="-43.18" y="-17.78"/>
 <wire x1="-43.18" y1="-17.78" x2="-38.1" y2="-17.78" width="0.1524" layer="91"/>
-<wire x1="45.72" y1="-22.86" x2="45.72" y2="-21.59" width="0.1524" layer="91"/>
-<wire x1="45.72" y1="-21.59" x2="45.72" y2="-12.7" width="0.1524" layer="91"/>
-<wire x1="45.72" y1="-12.7" x2="35.56" y2="-12.7" width="0.1524" layer="91"/>
+<wire x1="50.8" y1="-12.7" x2="45.72" y2="-12.7" width="0.1524" layer="91"/>
 <junction x="35.56" y="-12.7"/>
 <pinref part="GND2" gate="1" pin="GND"/>
-<wire x1="50.8" y1="-12.7" x2="45.72" y2="-12.7" width="0.1524" layer="91"/>
+<pinref part="D12" gate="1" pin="C"/>
+<wire x1="45.72" y1="-12.7" x2="35.56" y2="-12.7" width="0.1524" layer="91"/>
+<wire x1="45.72" y1="-20.32" x2="45.72" y2="-12.7" width="0.1524" layer="91"/>
 <junction x="45.72" y="-12.7"/>
-<pinref part="D12" gate="1" pin="A"/>
-<junction x="45.72" y="-21.59"/>
 </segment>
 <segment>
@@
 </sheet>
 </sheets>
+<errors>
+</errors>
 </schematic>
 </drawing>
